File: TiLDA Mk2 Prototype.sch (EAGLE design)
At the start: 0 parts

Commit message: Prototype: Working on board outline and initial layout
Parts:
- added H1: MOUNT-HOLE5.0, holes:MOUNT-HOLE5.0
- added J1: SPARKFUN_AVR_SPI_PRG_6NS, TiLDA Mk2 Parts:SPARKFUN_AVR_SPI_PRG_6NS
- added JP1, JP2, JP3: FIDUCIAL1X2.5-STOP, TiLDA Mk2 Parts:FIDUCIAL1X2.5-STOP
- added LOGO1: OSHW-LOGOM, TiLDA Mk2 Parts:OSHW-LOGOM
- added LOGO2: EMFLOGO-BOTH, TiLDA Mk2 Parts:EMFLOGO-BOTH
- added LOGO3: CISECOLOGO-LARGE, TiLDA Mk2 Parts:CISECOLOGO-LARGE
- added U$1: EPD-OUTLINE-2.7", TiLDA Mk2 Parts:EPD-OUTLINE-2.7"
- added U$2: TILDA_BOARDOUTLINE, TiLDA Mk2 Parts:TILDA_BOARDOUTLINE
- added U$3: SRF-LANDING-1.0A-MOVE, Ciseco Footprints:SRF-LANDING-1.0A-MOVE
- added U1: ATSAM3X8EA-AU, SmartPrj:ATSAM3X/AAU
- added U2: MPU-6000QFN-24, TiLDA Mk2 Parts:MPU-6000QFN-24
- added U3: ARDUINOR3-CISECO, TiLDA Mk2 Parts:ARDUINOR3-CISECO
- added USB1: SERIAL_MICRO-USB-ZX62-B-5PA, TiLDA Mk2 Parts:SERIAL_MICRO-USB-ZX62-B-5PA
- added X1: 52745-3090, con-molex:52745-3090
