File: TiLDA Mk2 Prototype v0.1.sch (EAGLE design)
At the start: 199 parts, among them IC1 ATSAM3X8EA-AU, IC10 MCP73831, IC2 MPU-6050, IC3 SRF-V1.2, IC5 S25FL216K0PMFI011, IC7 HMC5883LSMD (NP), IC8 MCP1825T-3302E/DC, IC9 TC1015-3V3, J1 ZX62-AB-5PA(11), J3 Arduino Headers, J5 1050270001 (NP), J6 B016 - PowerPOD NCP1402 5V0, J7 SFV30R-2STE1HLF, J8 1x02 RA Pin, Q10 2N7002KW, Q11 BSS84W, Q12 2N7002KW, Q13 BSS84W, Q8 BSS84W, Q9 2N7002KW, U2 JHD12864-G13BSW-OUTLINE, X1 12Mhz 13pF 30ppm (7pf caps), X2 32.768Khz

Commit message: Parts: Joystick footprint Prototype: Joystick footprint
Parts:
- S7: device TiLDA Mk2 Parts:JOYSTICK_MINI-APLS -> TiLDA Mk2 Parts:JOYSTICK_MINI_MULTICOMP
Changed lines of the file:
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@@
 <part name="GND47" library="TiLDA Mk2 Parts" deviceset="GND" device=""/>
 <part name="GND48" library="TiLDA Mk2 Parts" deviceset="GND" device=""/>
-<part name="S7" library="TiLDA Mk2 Parts" deviceset="JOYSTICK_MINI" device="-APLS" value="SKRHAAE010"/>
+<part name="S7" library="TiLDA Mk2 Parts" deviceset="JOYSTICK_MINI" device="_MULTICOMP" value="SKRHAAE010"/>
 <part name="SJ5" library="TiLDA Mk2 Parts" deviceset="SOLDERJUMPER_2WAY" device="S" value="RESET SELECT"/>
 <part name="R21" library="TiLDA Mk2 Parts" deviceset="R-EU_" device="R0402-ARDUINO-ROUND" value="0402/100K/1%"/>

Commit message: Prototype: 0805 LED's
Parts:
- removed LOGO2: EMFLOGO-SYMBOL, TiLDA Mk2 Parts:EMFLOGO-SYMBOL
- RX, TX: device TiLDA Mk2 Parts:LED0603-CORRECT -> TiLDA Mk2 Parts:LED0805-CORRECT
Changed lines of the file:
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@@
 <layer number="35" name="tGlue" color="7" fill="4" visible="no" active="no"/>
 <layer number="36" name="bGlue" color="7" fill="5" visible="no" active="no"/>
-<layer number="37" name="tTest" color="7" fill="1" visible="no" active="no"/>
-<layer number="38" name="bTest" color="7" fill="1" visible="no" active="no"/>
+<layer number="37" name="tTest" color="7" fill="1" visible="yes" active="no"/>
+<layer number="38" name="bTest" color="7" fill="1" visible="yes" active="no"/>
 <layer number="39" name="tKeepout" color="4" fill="11" visible="no" active="no"/>
 <layer number="40" name="bKeepout" color="1" fill="11" visible="no" active="no"/>
@@
 <layer number="44" name="Drills" color="7" fill="1" visible="no" active="no"/>
 <layer number="45" name="Holes" color="7" fill="1" visible="no" active="no"/>
-<layer number="46" name="Milling" color="3" fill="1" visible="no" active="no"/>
-<layer number="47" name="Measures" color="7" fill="1" visible="no" active="no"/>
-<layer number="48" name="Document" color="7" fill="1" visible="no" active="no"/>
-<layer number="49" name="Reference" color="13" fill="1" visible="no" active="no"/>
-<layer number="50" name="dxf" color="7" fill="1" visible="no" active="no"/>
-<layer number="51" name="tDocu" color="14" fill="1" visible="no" active="no"/>
-<layer number="52" name="bDocu" color="7" fill="1" visible="no" active="no"/>
-<layer number="53" name="tGND_GNDA" color="7" fill="9" visible="no" active="no"/>
-<layer number="54" name="bGND_GNDA" color="1" fill="9" visible="no" active="no"/>
-<layer number="56" name="wert" color="7" fill="1" visible="no" active="no"/>
-<layer number="57" name="tCAD" color="7" fill="1" visible="no" active="no"/>
+<layer number="46" name="Milling" color="3" fill="1" visible="yes" active="no"/>
+<layer number="47" name="Measures" color="7" fill="1" visible="yes" active="no"/>
+<layer number="48" name="Document" color="7" fill="1" visible="yes" active="no"/>
+<layer number="49" name="Reference" color="13" fill="1" visible="yes" active="no"/>
+<layer number="50" name="dxf" color="7" fill="1" visible="yes" active="no"/>
+<layer number="51" name="tDocu" color="14" fill="1" visible="yes" active="no"/>
+<layer number="52" name="bDocu" color="7" fill="1" visible="yes" active="no"/>
+<layer number="53" name="tGND_GNDA" color="7" fill="9" visible="yes" active="no"/>
+<layer number="54" name="bGND_GNDA" color="1" fill="9" visible="yes" active="no"/>
+<layer number="56" name="wert" color="7" fill="1" visible="yes" active="no"/>
+<layer number="57" name="tCAD" color="7" fill="1" visible="yes" active="no"/>
 <layer number="91" name="Nets" color="2" fill="1" visible="yes" active="yes"/>
 <layer number="92" name="Busses" color="1" fill="1" visible="yes" active="yes"/>
@@
 <part name="FID2" library="TiLDA Mk2 Parts" deviceset="FIDUCIAL" device="1X2.5-STOP"/>
 <part name="FID4" library="TiLDA Mk2 Parts" deviceset="FIDUCIAL" device="1X2.5-STOP"/>
-<part name="LOGO2" library="TiLDA Mk2 Parts" deviceset="EMFLOGO" device="-SYMBOL"/>
 <part name="IC3" library="Ciseco Footprints" deviceset="SRF" device="-LANDING-1.2" value="SRF-V1.2"/>
 <part name="X1" library="TiLDA Mk2 Parts" deviceset="CRYSTAL" device="-5X3.2" value="12Mhz 13pF 30ppm (7pf caps)"/>
@@
 <part name="GND35" library="TiLDA Mk2 Parts" deviceset="GND" device=""/>
 <part name="GND36" library="TiLDA Mk2 Parts" deviceset="GND" device=""/>
-<part name="TX" library="TiLDA Mk2 Parts" deviceset="LED" device="0603-CORRECT" value="0603/LED/RED"/>
-<part name="RX" library="TiLDA Mk2 Parts" deviceset="LED" device="0603-CORRECT" value="0603/LED/RED"/>
+<part name="TX" library="TiLDA Mk2 Parts" deviceset="LED" device="0805-CORRECT" value="0603/LED/RED"/>
+<part name="RX" library="TiLDA Mk2 Parts" deviceset="LED" device="0805-CORRECT" value="0603/LED/RED"/>
 <part name="R105" library="TiLDA Mk2 Parts" deviceset="R-EU_" device="R0402-ARDUINO-ROUND" value="0402/39R/1%"/>
 <part name="R106" library="TiLDA Mk2 Parts" deviceset="R-EU_" device="R0402-ARDUINO-ROUND" value="0402/39R/1%"/>
@@
 <instance part="FID2" gate="G$1" x="350.52" y="22.86"/>
 <instance part="FID4" gate="G$1" x="355.6" y="22.86"/>
-<instance part="LOGO2" gate="G$1" x="690.88" y="2.54"/>
 <instance part="IC3" gate="G$1" x="170.18" y="200.66"/>
 <instance part="X1" gate="G$1" x="477.52" y="198.12" smashed="yes" rot="R90">

Commit message: Prototype: Minor tweaks, adding TP27, moved L102, L105
Parts:
- added TP27: PB10, TiLDA Mk2 Parts:TPB1,27
Connections:
- net LCD_CS renamed LCD_!CS
- net PB18 renamed A63
- net PB19 renamed A64
- net PC12 renamed D51
- net PC3 renamed D35
- net UOTGVBOF: now also TP27.TP
Other:
- note added: "Light"
- note added: "SRF_P2_0/AT_COMMAND"
- note added: "TP27 for UOTGVBOF"
Changed lines of the file:
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@@
 <grid distance="0.1" unitdist="inch" unit="inch" style="lines" multiple="1" display="no" altdistance="0.01" altunitdist="inch" altunit="inch"/>
 <layers>
-<layer number="1" name="Top" color="4" fill="1" visible="yes" active="no"/>
-<layer number="2" name="Route2" color="1" fill="3" visible="yes" active="no"/>
-<layer number="3" name="Route3" color="4" fill="3" visible="yes" active="no"/>
-<layer number="4" name="Route4" color="1" fill="4" visible="yes" active="no"/>
-<layer number="5" name="Route5" color="4" fill="4" visible="yes" active="no"/>
-<layer number="6" name="Route6" color="1" fill="8" visible="yes" active="no"/>
-<layer number="7" name="Route7" color="4" fill="8" visible="yes" active="no"/>
-<layer number="8" name="Route8" color="1" fill="2" visible="yes" active="no"/>
-<layer number="9" name="Route9" color="4" fill="2" visible="yes" active="no"/>
-<layer number="10" name="Route10" color="1" fill="7" visible="yes" active="no"/>
-<layer number="11" name="Route11" color="4" fill="7" visible="yes" active="no"/>
-<layer number="12" name="Route12" color="1" fill="5" visible="yes" active="no"/>
-<layer number="13" name="Route13" color="4" fill="5" visible="yes" active="no"/>
-<layer number="14" name="Route14" color="1" fill="6" visible="yes" active="no"/>
-<layer number="15" name="Route15" color="4" fill="6" visible="yes" active="no"/>
-<layer number="16" name="Bottom" color="1" fill="1" visible="yes" active="no"/>
-<layer number="17" name="Pads" color="2" fill="1" visible="yes" active="no"/>
-<layer number="18" name="Vias" color="2" fill="1" visible="yes" active="no"/>
-<layer number="19" name="Unrouted" color="6" fill="1" visible="yes" active="no"/>
-<layer number="20" name="Dimension" color="15" fill="1" visible="yes" active="no"/>
-<layer number="21" name="tPlace" color="7" fill="1" visible="yes" active="no"/>
-<layer number="22" name="bPlace" color="6" fill="1" visible="yes" active="no"/>
-<layer number="23" name="tOrigins" color="15" fill="1" visible="yes" active="no"/>
-<layer number="24" name="bOrigins" color="15" fill="1" visible="yes" active="no"/>
-<layer number="25" name="tNames" color="7" fill="1" visible="yes" active="no"/>
-<layer number="26" name="bNames" color="7" fill="1" visible="yes" active="no"/>
-<layer number="27" name="tValues" color="7" fill="1" visible="yes" active="no"/>
-<layer number="28" name="bValues" color="7" fill="1" visible="yes" active="no"/>
+<layer number="1" name="Top" color="4" fill="1" visible="no" active="no"/>
+<layer number="2" name="Route2" color="1" fill="3" visible="no" active="no"/>
+<layer number="3" name="Route3" color="4" fill="3" visible="no" active="no"/>
+<layer number="4" name="Route4" color="1" fill="4" visible="no" active="no"/>
+<layer number="5" name="Route5" color="4" fill="4" visible="no" active="no"/>
+<layer number="6" name="Route6" color="1" fill="8" visible="no" active="no"/>
+<layer number="7" name="Route7" color="4" fill="8" visible="no" active="no"/>
+<layer number="8" name="Route8" color="1" fill="2" visible="no" active="no"/>
+<layer number="9" name="Route9" color="4" fill="2" visible="no" active="no"/>
+<layer number="10" name="Route10" color="1" fill="7" visible="no" active="no"/>
+<layer number="11" name="Route11" color="4" fill="7" visible="no" active="no"/>
+<layer number="12" name="Route12" color="1" fill="5" visible="no" active="no"/>
+<layer number="13" name="Route13" color="4" fill="5" visible="no" active="no"/>
+<layer number="14" name="Route14" color="1" fill="6" visible="no" active="no"/>
+<layer number="15" name="Route15" color="4" fill="6" visible="no" active="no"/>
+<layer number="16" name="Bottom" color="1" fill="1" visible="no" active="no"/>
+<layer number="17" name="Pads" color="2" fill="1" visible="no" active="no"/>
+<layer number="18" name="Vias" color="2" fill="1" visible="no" active="no"/>
+<layer number="19" name="Unrouted" color="6" fill="1" visible="no" active="no"/>
+<layer number="20" name="Dimension" color="15" fill="1" visible="no" active="no"/>
+<layer number="21" name="tPlace" color="7" fill="1" visible="no" active="no"/>
+<layer number="22" name="bPlace" color="6" fill="1" visible="no" active="no"/>
+<layer number="23" name="tOrigins" color="15" fill="1" visible="no" active="no"/>
+<layer number="24" name="bOrigins" color="15" fill="1" visible="no" active="no"/>
+<layer number="25" name="tNames" color="7" fill="1" visible="no" active="no"/>
+<layer number="26" name="bNames" color="7" fill="1" visible="no" active="no"/>
+<layer number="27" name="tValues" color="7" fill="1" visible="no" active="no"/>
+<layer number="28" name="bValues" color="7" fill="1" visible="no" active="no"/>
 <layer number="29" name="tStop" color="7" fill="3" visible="no" active="no"/>
 <layer number="30" name="bStop" color="7" fill="6" visible="no" active="no"/>
@@
 <layer number="35" name="tGlue" color="7" fill="4" visible="no" active="no"/>
 <layer number="36" name="bGlue" color="7" fill="5" visible="no" active="no"/>
-<layer number="37" name="tTest" color="7" fill="1" visible="yes" active="no"/>
-<layer number="38" name="bTest" color="7" fill="1" visible="yes" active="no"/>
+<layer number="37" name="tTest" color="7" fill="1" visible="no" active="no"/>
+<layer number="38" name="bTest" color="7" fill="1" visible="no" active="no"/>
 <layer number="39" name="tKeepout" color="4" fill="11" visible="no" active="no"/>
 <layer number="40" name="bKeepout" color="1" fill="11" visible="no" active="no"/>
@@
 <layer number="44" name="Drills" color="7" fill="1" visible="no" active="no"/>
 <layer number="45" name="Holes" color="7" fill="1" visible="no" active="no"/>
-<layer number="46" name="Milling" color="3" fill="1" visible="yes" active="no"/>
-<layer number="47" name="Measures" color="7" fill="1" visible="yes" active="no"/>
-<layer number="48" name="Document" color="7" fill="1" visible="yes" active="no"/>
-<layer number="49" name="Reference" color="13" fill="1" visible="yes" active="no"/>
-<layer number="50" name="dxf" color="7" fill="1" visible="yes" active="no"/>
-<layer number="51" name="tDocu" color="14" fill="1" visible="yes" active="no"/>
-<layer number="52" name="bDocu" color="7" fill="1" visible="yes" active="no"/>
-<layer number="53" name="tGND_GNDA" color="7" fill="9" visible="yes" active="no"/>
-<layer number="54" name="bGND_GNDA" color="1" fill="9" visible="yes" active="no"/>
-<layer number="56" name="wert" color="7" fill="1" visible="yes" active="no"/>
-<layer number="57" name="tCAD" color="7" fill="1" visible="yes" active="no"/>
+<layer number="46" name="Milling" color="3" fill="1" visible="no" active="no"/>
+<layer number="47" name="Measures" color="7" fill="1" visible="no" active="no"/>
+<layer number="48" name="Document" color="7" fill="1" visible="no" active="no"/>
+<layer number="49" name="Reference" color="13" fill="1" visible="no" active="no"/>
+<layer number="50" name="dxf" color="7" fill="1" visible="no" active="no"/>
+<layer number="51" name="tDocu" color="14" fill="1" visible="no" active="no"/>
+<layer number="52" name="bDocu" color="7" fill="1" visible="no" active="no"/>
+<layer number="53" name="tGND_GNDA" color="7" fill="9" visible="no" active="no"/>
+<layer number="54" name="bGND_GNDA" color="1" fill="9" visible="no" active="no"/>
+<layer number="56" name="wert" color="7" fill="1" visible="no" active="no"/>
+<layer number="57" name="tCAD" color="7" fill="1" visible="no" active="no"/>
 <layer number="91" name="Nets" color="2" fill="1" visible="yes" active="yes"/>
 <layer number="92" name="Busses" color="1" fill="1" visible="yes" active="yes"/>
@@
 <part name="GND9" library="TiLDA Mk2 Parts" deviceset="GND" device=""/>
 <part name="Q12" library="TiLDA Mk2 Parts" deviceset="MOSFET-N" device="SC70-3" value="2N7002KW"/>
+<part name="TP27" library="TiLDA Mk2 Parts" deviceset="TP" device="B1,27" value="PB10">
+<attribute name="TP_SIGNAL_NAME" value=""/>
+</part>
 </parts>
 <sheets>
@@
 <text x="800.1" y="132.08" size="1.778" layer="91">Off posotion power is taken from USB</text>
 <text x="800.1" y="129.54" size="1.778" layer="91">Battery is charged in both cases</text>
+<text x="797.56" y="127" size="1.778" layer="91">TP27 for UOTGVBOF</text>
+<text x="474.98" y="142.24" size="1.778" layer="91">Light</text>
+<text x="477.52" y="99.06" size="1.778" layer="91">SRF_P2_0/AT_COMMAND</text>
 </plain>
 <instances>
@@
 <instance part="GND9" gate="1" x="91.44" y="38.1"/>
 <instance part="Q12" gate="G$1" x="60.96" y="220.98" rot="MR270"/>
+<instance part="TP27" gate="G$1" x="563.88" y="45.72" rot="R180"/>
 </instances>
 <busses>
 </busses>
 <nets>
-<net name="LCD_CS" class="0">
+<net name="LCD_!CS" class="0">
 <segment>
 <pinref part="IC1" gate="G$1" pin="PB21"/>
@@
 <segment>
 <pinref part="IC1" gate="G$1" pin="PB10"/>
-<wire x1="563.88" y1="63.5" x2="563.88" y2="66.04" width="0.1524" layer="91"/>
 <label x="563.88" y="63.5" size="1.778" layer="95" rot="MR270"/>
+<pinref part="TP27" gate="G$1" pin="TP"/>
+<wire x1="563.88" y1="48.26" x2="563.88" y2="66.04" width="0.1524" layer="91"/>
 </segment>
 </net>
@@
 </segment>
 </net>
-<net name="PB19" class="0">
+<net name="A64" class="0">
 <segment>
 <pinref part="IC1" gate="G$1" pin="PB19"/>
@@
 </segment>
 </net>
-<net name="PB18" class="0">
+<net name="A63" class="0">
 <segment>
 <pinref part="IC1" gate="G$1" pin="PB18"/>
@@
 </segment>
 </net>
-<net name="PC12" class="0">
+<net name="D51" class="0">
 <segment>
 <pinref part="IC1" gate="G$1" pin="PC12"/>
@@
 </segment>
 </net>
-<net name="PC3" class="0">
+<net name="D35" class="0">
 <segment>
 <pinref part="IC1" gate="G$1" pin="PC3"/>

Commit message: Prototype: Get backlight onto a PWM, swapped LCD_BACKLIGHT and TP25.
Parts:
- TP25: value PC3 -> PC1
Connections:
- removed net D35: IC1.PC3, TP25.TP
- new net D33: IC1.PC1, TP25.TP
- net LCD_BACKLIGHT: now also IC1.PC3; no longer IC1.PC1
Other:
- moved on the sheet: TP25
Changed lines of the file:
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@@
 </part>
 <part name="SJ10" library="TiLDA Mk2 Parts" deviceset="SOLDERJUMPER_2WAY" device="S" value="VDDIO"/>
-<part name="TP25" library="TiLDA Mk2 Parts" deviceset="TP" device="B1,27" value="PC3">
+<part name="TP25" library="TiLDA Mk2 Parts" deviceset="TP" device="B1,27" value="PC1">
 <attribute name="TP_SIGNAL_NAME" value=""/>
 </part>
@@
 <instance part="TP23" gate="G$1" x="586.74" y="45.72" rot="R180"/>
 <instance part="SJ10" gate="G$1" x="568.96" y="223.52" rot="R90"/>
-<instance part="TP25" gate="G$1" x="673.1" y="83.82" rot="R270"/>
+<instance part="TP25" gate="G$1" x="673.1" y="78.74" rot="R270"/>
 <instance part="TP26" gate="G$1" x="670.56" y="182.88" rot="R270"/>
 <instance part="J6" gate="G$1" x="88.9" y="144.78"/>
@@
 </segment>
 <segment>
-<pinref part="IC1" gate="G$1" pin="PC1"/>
-<wire x1="637.54" y1="78.74" x2="635" y2="78.74" width="0.1524" layer="91"/>
-<label x="637.54" y="78.74" size="1.778" layer="95"/>
+<pinref part="IC1" gate="G$1" pin="PC3"/>
+<label x="637.54" y="83.82" size="1.778" layer="95"/>
+<wire x1="637.54" y1="83.82" x2="635" y2="83.82" width="0.1524" layer="91"/>
 </segment>
 </net>
@@
 </segment>
 </net>
-<net name="D35" class="0">
-<segment>
-<pinref part="IC1" gate="G$1" pin="PC3"/>
-<label x="647.7" y="83.82" size="1.778" layer="95"/>
-<pinref part="TP25" gate="G$1" pin="TP"/>
-<wire x1="670.56" y1="83.82" x2="635" y2="83.82" width="0.1524" layer="91"/>
-</segment>
-</net>
 <net name="N$1" class="0">
 <segment>
@@
 </segment>
 </net>
+<net name="D33" class="0">
+<segment>
+<pinref part="IC1" gate="G$1" pin="PC1"/>
+<wire x1="670.56" y1="78.74" x2="635" y2="78.74" width="0.1524" layer="91"/>
+<label x="647.7" y="78.74" size="1.778" layer="95"/>
+<pinref part="TP25" gate="G$1" pin="TP"/>
+</segment>
+</net>

Commit message: Prototype: Get LIGHT on to a wake up pin, swapped LIGTH with AT_COMMAND
Connections:
- net LIGHT: now also IC1.PA3; no longer IC1.PA20
- net SRF_P2_0/AT_COMMAND: now also IC1.PA20; no longer IC1.PA3
Other:
- note removed: "Light"
- note removed: "SRF_P2_0/AT_COMMAND"
Changed lines of the file:
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@@
 <text x="800.1" y="129.54" size="1.778" layer="91">Battery is charged in both cases</text>
 <text x="797.56" y="127" size="1.778" layer="91">TP27 for UOTGVBOF</text>
-<text x="474.98" y="142.24" size="1.778" layer="91">Light</text>
-<text x="477.52" y="99.06" size="1.778" layer="91">SRF_P2_0/AT_COMMAND</text>
 </plain>
 <instances>
@@
 </segment>
 <segment>
-<pinref part="IC1" gate="G$1" pin="PA20"/>
-<wire x1="513.08" y1="99.06" x2="515.62" y2="99.06" width="0.1524" layer="91"/>
-<label x="513.08" y="99.06" size="1.778" layer="95" rot="MR0"/>
+<pinref part="IC1" gate="G$1" pin="PA3"/>
+<wire x1="515.62" y1="142.24" x2="513.08" y2="142.24" width="0.1524" layer="91"/>
+<label x="513.08" y="142.24" size="1.778" layer="95" rot="MR0"/>
 </segment>
 </net>
@@
 </segment>
 <segment>
-<pinref part="IC1" gate="G$1" pin="PA3"/>
-<wire x1="515.62" y1="142.24" x2="513.08" y2="142.24" width="0.1524" layer="91"/>
-<label x="513.08" y="142.24" size="1.778" layer="95" rot="MR0"/>
+<pinref part="IC1" gate="G$1" pin="PA20"/>
+<wire x1="513.08" y1="99.06" x2="515.62" y2="99.06" width="0.1524" layer="91"/>
+<label x="513.08" y="99.06" size="1.778" layer="95" rot="MR0"/>
 </segment>
 </net>

Commit message: Prototype: VDDIO rewire
Connections:
- removed net N$11: R8.1, TX.A
- removed net N$13: R14.1, RX.A
- new net N$2: R8.1, TX.C
- new net N$3: R14.1, RX.C
- new net VDDIO: C101.+, C104.2, C105.2, C107.2, C108.2, C118.2, IC1.VDDIO1, IC1.VDDIO2, IC1.VDDIO3, IC1.VDDIO4, L101.1, L102.1, R21.2, R22.2, R23.2, R24.2, R44.2, R47.2, R48.2, R49.1, SJ10.2, SJ8.3
- net 3V3: no longer C101.+, C104.2, C105.2, C107.2, C108.2, C118.2, IC1.VDDIO1, IC1.VDDIO2, IC1.VDDIO3, IC1.VDDIO4, L101.1, L102.1, R14.2, R21.2, R22.2, R23.2, R24.2, R44.2, R49.1, R8.2, SJ10.2, SJ8.3
- net GND: now also R14.2, R8.2
- net RXL: now also RX.A; no longer RX.C
- net TXL: now also TX.A; no longer TX.C
- net VBACKUP: no longer R47.2, R48.2
Other:
- moved on the sheet: R49, RX, TX
